File: pcbs/calico/calico.kicad_sch (KiCad schematic)
At the start: 61 parts, among them J1 MJ-4PP-9-kbd-corne-light-resc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, SW1 SW_Push, SW10 SW_Push, SW11 SW_Push, SW12 SW_Push, SW13 SW_Push, SW14 SW_Push, SW15 SW_Push, SW16 SW_Push, SW17 SW_Push, SW18 SW_Push, SW19 SW_Push, SW2 SW_Push, SW20 SW_Push, SW21 SW_Push, SW22 SW_Push, SW23 SW_Push, SW24 SW_Push, SW25 SW_Push, SW26 SW_Push, SW27 SW_Push, SW3 SW_Push, SW4 SW_Push, SW5 SW_Push, SW6 SW_Push, SW7 SW_Push, SW8 SW_Push, SW9 SW_Push

Commit message: v0.2 initial
Parts:
- J1: footprint calico:TRRS-3pin -> calico:TRRS-3pin_modified
- RSW1: footprint calico:Reset -> calico:Reset_modified
- U1: footprint tree:ProMicro -> calico:ProMicro_jumpers
Changed lines of the file:
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@@
 			)
 		)
-		(property "Footprint" "tree:ProMicro"
+		(property "Footprint" "calico:ProMicro_jumpers"
 			(at 209.55 38.1 0)
 			(effects
@@
 			)
 		)
-		(property "Footprint" "calico:TRRS-3pin"
+		(property "Footprint" "calico:TRRS-3pin_modified"
 			(at 217.805 92.075 0)
 			(effects
@@
 			)
 		)
-		(property "Footprint" "calico:Reset"
+		(property "Footprint" "calico:Reset_modified"
 			(at 259.08 39.37 0)
 			(effects
